File: Électrique/Clavier/Clavier_drive_1/Clavier_drive_1.kicad_pcb (KiCad board)
At the start: 2 copper layers, 177 parts, among them IC12 TCAN332DR, IC3 TLV1117-33IDCY, J10 Conn_01x02_Pin, J16 B5B-XH-A_LF__SN_, J9 Conn_01x02_Pin, SW15 Switch, SW16 Switch, SW17 Switch, SW18 Switch, SW19 Switch, SW20 Switch, SW23 Switch, SW24 Switch, SW25 Switch, SW26 Switch, SW27 Switch, SW28 Switch, SW29 Switch, SW30 Switch, SW31 Switch, SW32 Switch, SW33 Switch, SW34 Switch, SW35 Switch, SW36 Switch, SW37 Switch, SW38 Switch, SW39 Switch, SW40 Switch, SW41 Switch, SW42 Switch, SW43 Switch, SW44 Switch, SW45 Switch, SW46 Switch, SW47 Switch, SW48 Switch, SW51 Switch, SW52 Switch, SW53 Switch, SW54 Switch, SW55 Switch, SW56 Switch, SW57 Switch, SW58 Switch, SW59 Switch, SW60 Switch, SW61 Switch, SW62 Switch, SW63 Switch, SW64 Switch, SW65 Switch, SW66 Switch, SW67 Switch, SW68 Switch, SW69 Switch, SW70 Switch, SW71 Switch, SW72 Switch, SW73 Switch, SW74 Switch, SW75 Switch, SW76 Switch, SW79 Switch, SW80 Switch, SW81 Switch, SW82 Switch, SW83 Switch, SW84 Switch, SW86 Switch, SW87 Switch, SW88 Switch, SW89 Switch, SW90 Switch, SW91 Switch, SW92 Switch, SW93 Switch, SW94 Switch, SW95 Switch

Commit message: ajout firmware + modif readme
Parts:
- removed D1, D2, D3, D35, D36, D4, D5, D6, D63, D64, D7: 1N4148W, Diode_SMD:D_SOD-123
- removed J10, J9: Conn_01x02_Pin, SamacSys:SHDRRA2W50P0X200_1X2_600X770X525P
- removed J16: B5B-XH-A_LF__SN_, SamacSys:SHDR5W64P0X250_1X5_1490X575X700P
- removed S2, S3, S4, S5, S6, S7: MTS-103, switchboard:MTS-103 Switch
- removed SW35, SW36, SW63, SW64: Switch, PCM_marbastlib-mx:SW_MX_HS_CPG151101S11_1u
- added C101: CL31A476MPHNNNE, SamacSys:CAPC3216X180N, B.Cu at (98.4, 54.0)
- added C102: CL31A476MPHNNNE, SamacSys:CAPC3216X180N, B.Cu at (96.1, 53.6)
- added C103: 0.1uF, Capacitor_SMD:C_0402_1005Metric, B.Cu at (98.3, 60.1)
- added C104: 0.1uF, Capacitor_SMD:C_0402_1005Metric, B.Cu at (98.7, 58.1)
- added C105: 0.1uF, Capacitor_SMD:C_0402_1005Metric, B.Cu at (109.0, 77.2)
- added C106: 0.1uF, Capacitor_SMD:C_0402_1005Metric, B.Cu at (109.0, 81.8)
- added C107: 0.1uF, Capacitor_SMD:C_0402_1005Metric, B.Cu at (109.0, 86.5)
- added C108: 0.1uF, Capacitor_SMD:C_0402_1005Metric, B.Cu at (109.0, 58.2)
- added C109: 0.1uF, Capacitor_SMD:C_0402_1005Metric, B.Cu at (187.1, 59.7)
- added C110: 0.1uF, Capacitor_SMD:C_0402_1005Metric, B.Cu at (187.9, 64.2)
- added C111: 0.1uF, Capacitor_SMD:C_0402_1005Metric, B.Cu at (162.8, 66.5)
- added C112: 0.1uF, Capacitor_SMD:C_0402_1005Metric, B.Cu at (162.8, 81.0)
- added C113: 0.1uF, Capacitor_SMD:C_0402_1005Metric, B.Cu at (162.8, 104.7)
- added C114: 0.1uF, Capacitor_SMD:C_0402_1005Metric, B.Cu at (162.8, 100.2)
- added C115: 0.1uF, Capacitor_SMD:C_0402_1005Metric, B.Cu at (162.8, 90.2)
- added C116: 0.1uF, Capacitor_SMD:C_0402_1005Metric, B.Cu at (162.8, 85.6)
- added C117: 0.1uF, Capacitor_SMD:C_0402_1005Metric, B.Cu at (162.8, 62.0)
- added C118: 0.1uF, Capacitor_SMD:C_0402_1005Metric, B.Cu at (162.8, 71.1)
- added C119: 0.1uF, Capacitor_SMD:C_0402_1005Metric, B.Cu at (162.8, 109.2)
- added C120: 0.1uF, Capacitor_SMD:C_0402_1005Metric, B.Cu at (162.8, 128.3)
- added C121: 0.1uF, Capacitor_SMD:C_0402_1005Metric, B.Cu at (162.8, 123.7)
- added C122: 0.1uF, Capacitor_SMD:C_0402_1005Metric, B.Cu at (162.8, 119.2)
- added C123: 0.1uF, Capacitor_SMD:C_0402_1005Metric, B.Cu at (109.0, 67.2)
- added C124: 0.1uF, Capacitor_SMD:C_0402_1005Metric, B.Cu at (109.0, 62.8)
- added C125: 0.1uF, Capacitor_SMD:C_0402_1005Metric, B.Cu at (86.1, 51.6)
- added C126: 0.1uF, Capacitor_SMD:C_0402_1005Metric, B.Cu at (85.3, 56.0)
- added C127: 0.1uF, Capacitor_SMD:C_0402_1005Metric, B.Cu at (84.6, 60.5)
- added C128: 0.1uF, Capacitor_SMD:C_0402_1005Metric, B.Cu at (186.3, 55.3)
- added C129: 0.1uF, Capacitor_SMD:C_0402_1005Metric, B.Cu at (157.0, 25.6)
- added C130: 0.1uF, Capacitor_SMD:C_0402_1005Metric, B.Cu at (161.8, 25.8)
- added C131: 0.1uF, Capacitor_SMD:C_0402_1005Metric, B.Cu at (167.7, 22.7)
- added C132: 0.1uF, Capacitor_SMD:C_0402_1005Metric, B.Cu at (172.6, 23.8)
- added C133: 0.1uF, Capacitor_SMD:C_0402_1005Metric, B.Cu at (109.0, 100.8)
- added C134: 0.1uF, Capacitor_SMD:C_0402_1005Metric, B.Cu at (109.0, 124.4)
- added C135: 0.1uF, Capacitor_SMD:C_0402_1005Metric, B.Cu at (109.0, 96.2)
- added C136: 0.1uF, Capacitor_SMD:C_0402_1005Metric, B.Cu at (109.0, 119.8)
- added C137: 0.1uF, Capacitor_SMD:C_0402_1005Metric, B.Cu at (109.0, 105.3)
- added C138: 0.1uF, Capacitor_SMD:C_0402_1005Metric, B.Cu at (109.0, 115.3)
- added C139: CL31A476MPHNNNE, SamacSys:CAPC3216X180N, B.Cu at (161.2, 56.0)
- added C140: CL31A476MPHNNNE, SamacSys:CAPC3216X180N, B.Cu at (161.2, 53.7)
- added C141: CL31A476MPHNNNE, SamacSys:CAPC3216X180N, B.Cu at (110.8, 53.8)
- added C142: CL31A476MPHNNNE, SamacSys:CAPC3216X180N, B.Cu at (110.8, 55.9)
- added C143: CL31A476MPHNNNE, SamacSys:CAPC3216X180N, B.Cu at (176.7, 64.6)
- added C144: CL31A476MPHNNNE, SamacSys:CAPC3216X180N, B.Cu at (178.9, 64.2)
- added C2: 22uF, Capacitor_SMD:C_1206_3216Metric, B.Cu at (86.6, 21.7)
- added D101: 1N4148W, Diode_SMD:D_SOD-123, B.Cu at (182.6, 21.7)
- added D102: 1N4148W, Diode_SMD:D_SOD-123, B.Cu at (89.3, 35.1)
- added D103: 1N4148W, Diode_SMD:D_SOD-123, B.Cu at (82.6, 72.7)
- added D105: 1N4148W, Diode_SMD:D_SOD-123, B.Cu at (123.0, 118.0)
- added D106: 1N4148W, Diode_SMD:D_SOD-123, B.Cu at (123.0, 99.0)
- added D107: 1N4148W, Diode_SMD:D_SOD-123, B.Cu at (123.0, 80.0)
- added D108: 1N4148W, Diode_SMD:D_SOD-123, B.Cu at (123.0, 61.0)
- added D109: 1N4148W, Diode_SMD:D_SOD-123, B.Cu at (142.0, 99.0)
- added D110: 1N4148W, Diode_SMD:D_SOD-123, B.Cu at (142.0, 80.0)
- added D111: 1N4148W, Diode_SMD:D_SOD-123, B.Cu at (142.0, 61.0)
- added D112: 1N4148W, Diode_SMD:D_SOD-123, B.Cu at (176.9, 36.8)
- added D113: 1N4148W, Diode_SMD:D_SOD-123, B.Cu at (183.4, 73.5)
- added D114: 1N4148W, Diode_SMD:D_SOD-123, B.Cu at (142.0, 118.0)
- added H101: MountingHole, MountingHole:MountingHole_3.2mm_M3_DIN965, F.Cu at (-11.8, 20.9)
- added H102: MountingHole, MountingHole:MountingHole_3.2mm_M3_DIN965, F.Cu at (-21.8, 77.2)
- added H103: MountingHole, MountingHole:MountingHole_3.2mm_M3_DIN965, F.Cu at (65.3, 22.3)
- added H104: MountingHole, MountingHole:MountingHole_3.2mm_M3_DIN965, F.Cu at (51.6, 100.3)
- added H105: MountingHole, MountingHole:MountingHole_3.2mm_M3_DIN965, F.Cu at (135.9, 74.1)
- added H106: MountingHole, MountingHole:MountingHole_3.2mm_M3_DIN965, F.Cu at (135.8, 112.2)
- added H107: MountingHole, MountingHole:MountingHole_3.2mm_M3_DIN965, F.Cu at (206.4, 22.3)
- added H108: MountingHole, MountingHole:MountingHole_3.2mm_M3_DIN965, F.Cu at (220.1, 100.3)
- added H109: MountingHole, MountingHole:MountingHole_3.2mm_M3_DIN965, F.Cu at (283.5, 20.9)
- added H110: MountingHole, MountingHole:MountingHole_3.2mm_M3_DIN965, F.Cu at (293.4, 77.2)
- added H111: MountingHole, MountingHole:MountingHole_3.2mm_M3_DIN965, F.Cu at (249.1, 45.3)
- added H112: MountingHole, MountingHole:MountingHole_3.2mm_M3_DIN965, F.Cu at (21.5, 51.3)
- added IC101: SN74LVC1T45DBVR, SamacSys:SOT95P280X145-6N, B.Cu at (95.9, 58.1)
- added IC102: SN74LVC1T45DBVR, SamacSys:SOT95P280X145-6N, B.Cu at (159.6, 23.7)
- added IC103: H11L1SR2VM, SamacSys:H11L1SR2VM, F.Cu at (181.9, 23.3)
- added IC104: SN74LVC1T45DBVR, SamacSys:SOT95P280X145-6N, B.Cu at (170.5, 21.8)
- added J101: SJ1-3533N, SamacSys:SJ13533N, F.Cu at (92.1, 5.17)
- added J102: SJ1-3533N, SamacSys:SJ13533N, F.Cu at (158.0, 8.98)
- added J103: SJ1-3533N, SamacSys:SJ13533N, F.Cu at (179.5, 5.17)
- added J104: SJ1-3533N, SamacSys:SJ13533N, F.Cu at (168.7, 7.08)
- added J105: SJ1-3533N, SamacSys:SJ13533N, F.Cu at (113.7, 8.98)
- added J106: SJ1-3533N, SamacSys:SJ13533N, F.Cu at (102.9, 7.08)
- added LED101: SK6812MINI-E, JANKO:LED-SMD_4P-L3.2-W2.8-LS5.9_SK6812MINI-E, B.Cu at (88.7, 53.9)
- added LED102: SK6812MINI-E, JANKO:LED-SMD_4P-L3.2-W2.8-LS5.9_SK6812MINI-E, B.Cu at (87.9, 58.4)
- added LED103: SK6812MINI-E, JANKO:LED-SMD_4P-L3.2-W2.8-LS5.9_SK6812MINI-E, B.Cu at (87.2, 62.8)
- added LED104: SK6812MINI-E, JANKO:LED-SMD_4P-L3.2-W2.8-LS5.9_SK6812MINI-E, B.Cu at (112.0, 60.0)
- added LED105: SK6812MINI-E, JANKO:LED-SMD_4P-L3.2-W2.8-LS5.9_SK6812MINI-E, B.Cu at (112.0, 64.6)
- added LED106: SK6812MINI-E, JANKO:LED-SMD_4P-L3.2-W2.8-LS5.9_SK6812MINI-E, B.Cu at (112.0, 69.2)
- added LED107: SK6812MINI-E, JANKO:LED-SMD_4P-L3.2-W2.8-LS5.9_SK6812MINI-E, B.Cu at (112.0, 79.1)
- added LED108: SK6812MINI-E, JANKO:LED-SMD_4P-L3.2-W2.8-LS5.9_SK6812MINI-E, B.Cu at (112.0, 83.7)
- added LED109: SK6812MINI-E, JANKO:LED-SMD_4P-L3.2-W2.8-LS5.9_SK6812MINI-E, B.Cu at (112.0, 88.2)
- added LED110: SK6812MINI-E, JANKO:LED-SMD_4P-L3.2-W2.8-LS5.9_SK6812MINI-E, B.Cu at (112.0, 98.2)
- added LED111: SK6812MINI-E, JANKO:LED-SMD_4P-L3.2-W2.8-LS5.9_SK6812MINI-E, B.Cu at (112.0, 102.7)
- added LED112: SK6812MINI-E, JANKO:LED-SMD_4P-L3.2-W2.8-LS5.9_SK6812MINI-E, B.Cu at (112.0, 107.2)
- added LED113: SK6812MINI-E, JANKO:LED-SMD_4P-L3.2-W2.8-LS5.9_SK6812MINI-E, B.Cu at (112.0, 117.2)
- added LED114: SK6812MINI-E, JANKO:LED-SMD_4P-L3.2-W2.8-LS5.9_SK6812MINI-E, B.Cu at (112.0, 121.8)
- added LED115: SK6812MINI-E, JANKO:LED-SMD_4P-L3.2-W2.8-LS5.9_SK6812MINI-E, B.Cu at (112.0, 126.3)
- added LED116: SK6812MINI-E, JANKO:LED-SMD_4P-L3.2-W2.8-LS5.9_SK6812MINI-E, B.Cu at (159.7, 126.3)
- added LED117: SK6812MINI-E, JANKO:LED-SMD_4P-L3.2-W2.8-LS5.9_SK6812MINI-E, B.Cu at (159.7, 121.8)
- added LED118: SK6812MINI-E, JANKO:LED-SMD_4P-L3.2-W2.8-LS5.9_SK6812MINI-E, B.Cu at (159.7, 117.2)
- added LED119: SK6812MINI-E, JANKO:LED-SMD_4P-L3.2-W2.8-LS5.9_SK6812MINI-E, B.Cu at (159.7, 107.2)
- added LED120: SK6812MINI-E, JANKO:LED-SMD_4P-L3.2-W2.8-LS5.9_SK6812MINI-E, B.Cu at (159.7, 102.7)
- added LED121: SK6812MINI-E, JANKO:LED-SMD_4P-L3.2-W2.8-LS5.9_SK6812MINI-E, B.Cu at (159.7, 98.2)
- added LED122: SK6812MINI-E, JANKO:LED-SMD_4P-L3.2-W2.8-LS5.9_SK6812MINI-E, B.Cu at (159.7, 88.2)
- added LED123: SK6812MINI-E, JANKO:LED-SMD_4P-L3.2-W2.8-LS5.9_SK6812MINI-E, B.Cu at (159.7, 83.7)
- added LED124: SK6812MINI-E, JANKO:LED-SMD_4P-L3.2-W2.8-LS5.9_SK6812MINI-E, B.Cu at (159.7, 79.1)
- added LED125: SK6812MINI-E, JANKO:LED-SMD_4P-L3.2-W2.8-LS5.9_SK6812MINI-E, B.Cu at (159.7, 69.2)
- added LED126: SK6812MINI-E, JANKO:LED-SMD_4P-L3.2-W2.8-LS5.9_SK6812MINI-E, B.Cu at (159.7, 64.6)
- added LED127: SK6812MINI-E, JANKO:LED-SMD_4P-L3.2-W2.8-LS5.9_SK6812MINI-E, B.Cu at (159.7, 60.0)
- added LED128: SK6812MINI-E, JANKO:LED-SMD_4P-L3.2-W2.8-LS5.9_SK6812MINI-E, B.Cu at (184.5, 62.8)
- added LED129: SK6812MINI-E, JANKO:LED-SMD_4P-L3.2-W2.8-LS5.9_SK6812MINI-E, B.Cu at (183.7, 58.4)
- added LED130: SK6812MINI-E, JANKO:LED-SMD_4P-L3.2-W2.8-LS5.9_SK6812MINI-E, B.Cu at (182.9, 53.9)
- added Q1: AO3401A, Package_TO_SOT_SMD:SOT-23, B.Cu at (150.1, 6.90)
- added R101: R510, Resistor_SMD:R_0603_1608Metric, B.Cu at (93.7, 54.8)
- added R102: R220, Resistor_SMD:R_0603_1608Metric, B.Cu at (160.4, 20.0)
- added R103: R220, Resistor_SMD:R_0603_1608Metric, B.Cu at (162.0, 19.7)
- added R104: R510, Resistor_SMD:R_0603_1608Metric, B.Cu at (181.9, 24.8)
- added R105: R220, Resistor_SMD:R_0603_1608Metric, B.Cu at (171.2, 18.1)
- added R106: R220, Resistor_SMD:R_0603_1608Metric, B.Cu at (182.6, 14.3)
- added R107: R220, Resistor_SMD:R_0603_1608Metric, B.Cu at (172.9, 17.8)
- added R33: R1K, Resistor_SMD:R_0603_1608Metric, B.Cu at (156.3, 36.5)
- added R34: 10k, Resistor_SMD:R_0603_1608Metric, B.Cu at (152.8, 29.4)
- added SW101: Switch, PCM_marbastlib-mx:SW_MX_HS_CPG151101S11_1u, B.Cu at (91.3, 39.6)
- added SW102: Switch, PCM_marbastlib-mx:SW_MX_HS_CPG151101S11_1u, B.Cu at (84.6, 77.1)
- added SW103: Switch, PCM_marbastlib-mx:SW_MX_HS_CPG151101S11_1u, B.Cu at (126.3, 121.8)
- added SW104: Switch, PCM_marbastlib-mx:SW_MX_HS_CPG151101S11_1u, B.Cu at (126.3, 102.7)
- added SW105: Switch, PCM_marbastlib-mx:SW_MX_HS_CPG151101S11_1u, B.Cu at (126.3, 83.7)
- added SW106: Switch, PCM_marbastlib-mx:SW_MX_HS_CPG151101S11_1u, B.Cu at (126.3, 64.6)
- added SW107: Switch, PCM_marbastlib-mx:SW_MX_HS_CPG151101S11_1u, B.Cu at (145.3, 102.7)
- added SW108: Switch, PCM_marbastlib-mx:SW_MX_HS_CPG151101S11_1u, B.Cu at (145.3, 83.7)
- added SW109: Switch, PCM_marbastlib-mx:SW_MX_HS_CPG151101S11_1u, B.Cu at (145.3, 64.6)
- added SW110: Switch, PCM_marbastlib-mx:SW_MX_HS_CPG151101S11_1u, B.Cu at (180.4, 39.6)
- added SW111: Switch, PCM_marbastlib-mx:SW_MX_HS_CPG151101S11_1u, B.Cu at (187.0, 77.1)
- added SW112: Switch, PCM_marbastlib-mx:SW_MX_HS_CPG151101S11_1u, B.Cu at (145.3, 121.8)
- C1, C10, C78, C8, C9, C99, D104, IC12, IC3, R24, TP2: moved to B.Cu
- S1: value MTS-103 -> TS-1088-AR02016; footprint switchboard:MTS-103 Switch -> SamacSys:TS1088AR02016
- moved C99 133.8 mm to (151.4, 29.7), turned to 90 degrees
- moved C1 132.3 mm to (103.7, 27.0), turned to -100 degrees
- moved C8 130.3 mm to (101.3, 24.6), turned to 80 degrees
- moved C9 126.8 mm to (89.3, 22.2), turned to -100 degrees
- moved C10 126.8 mm to (91.4, 21.5), turned to -100 degrees
- moved C78 124.7 mm to (118.0, 23.6), turned to -10 degrees
- moved IC3 116.9 mm to (96.0, 24.1), turned to -10 degrees
- moved TP2 111.5 mm to (104.3, 23.1), turned to -10 degrees
- moved IC12 107.9 mm to (113.2, 21.9), turned to 170 degrees
- moved R24 107.6 mm to (108.2, 19.0), turned to 170 degrees
- moved D104 105.0 mm to (97.0, 18.5), turned to -10 degrees
- moved A1 22.6 mm to (135.8, 29.7)
- moved D71 21.6 mm to (-35.5, 80.5)
- moved D20 21.2 mm to (73.5, 13.1)
- moved D34 21.2 mm to (70.2, 31.8)
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Connections:
- A1 pad 1: unconnected-(A1-GPIO0-Pad1) -> /RXD CAN
- A1 pad 10: unconnected-(A1-GPIO7-Pad10) -> /L2
- A1 pad 11: unconnected-(A1-GPIO8-Pad11) -> /L3
- A1 pad 12: unconnected-(A1-GPIO9-Pad12) -> /L4
- A1 pad 13: Net-(A1-GND-Pad13) -> GND
- A1 pad 15: unconnected-(A1-GPIO11-Pad15) -> /LED_DATA
- A1 pad 16: unconnected-(A1-GPIO12-Pad16) -> /C4
- A1 pad 17: unconnected-(A1-GPIO13-Pad17) -> /C3
- A1 pad 18: Net-(A1-GND-Pad13) -> GND
- A1 pad 19: unconnected-(A1-GPIO14-Pad19) -> /C2
- A1 pad 2: unconnected-(A1-GPIO1-Pad2) -> /TXD CAN
- A1 pad 20: unconnected-(A1-GPIO15-Pad20) -> /C1
- A1 pad 21: unconnected-(A1-GPIO16-Pad21) -> /C12
- A1 pad 22: unconnected-(A1-GPIO17-Pad22) -> /C11
- A1 pad 23: Net-(A1-GND-Pad13) -> GND
- A1 pad 24: unconnected-(A1-GPIO18-Pad24) -> /C10
- A1 pad 25: unconnected-(A1-GPIO19-Pad25) -> /C9
- A1 pad 26: unconnected-(A1-GPIO20-Pad26) -> /L7
- A1 pad 27: unconnected-(A1-GPIO21-Pad27) -> /L6
- A1 pad 28: Net-(A1-GND-Pad13) -> GND
- A1 pad 29: unconnected-(A1-GPIO22-Pad29) -> /L5
- A1 pad 3: Net-(A1-GND-Pad13) -> GND
- A1 pad 30: unconnected-(A1-RUN-Pad30) -> /RUN
- A1 pad 32: unconnected-(A1-GPIO27_ADC1-Pad32) -> /C8
- A1 pad 34: unconnected-(A1-GPIO28_ADC2-Pad34) -> /C7
- A1 pad 36: unconnected-(A1-3V3-Pad36) -> /3.3V RP
- A1 pad 38: Net-(A1-GND-Pad13) -> GND
- A1 pad 39: unconnected-(A1-VSYS-Pad39) -> Net-(A1-VSYS)
- A1 pad 4: unconnected-(A1-GPIO2-Pad4) -> /C6
- A1 pad 40: unconnected-(A1-VBUS-Pad40) -> Net-(A1-VBUS)
- A1 pad 5: unconnected-(A1-GPIO3-Pad5) -> /C5
- A1 pad 6: unconnected-(A1-GPIO4-Pad6) -> /TX PICO MIDI
- A1 pad 7: unconnected-(A1-GPIO5-Pad7) -> / RX PICO MIDI
- A1 pad 8: Net-(A1-GND-Pad13) -> GND
- A1 pad 9: unconnected-(A1-GPIO6-Pad9) -> /L1
- A1 pad D2: Net-(A1-GND-Pad13) -> GND
- C1 pad 1: 3.3VOUT -> 3.3VIN
- C8 pad 1: 3.3VOUT -> 3.3VIN
- D104 pad 2: 3.3VOUT -> 3.3VIN
- D43 pad 1: unconnected-(D43-K-Pad1) -> /L3
- D91 pad 1: /L5 -> /L6
- IC12 pad 1: /TXD -> /TXD CAN
- IC12 pad 4: /RXD -> /RXD CAN
- IC3 pad 2: 3.3VOUT -> 3.3VIN
- IC3 pad 4: 3.3VOUT -> 3.3VIN
- S1 pad 1: /C14 -> /RUN
- SW86 pad 1: /C3 -> /C2
- SW87 pad 1: /C4 -> /C3
- SW88 pad 1: /C5 -> /C4
- SW89 pad 1: /C6 -> /C5
- SW90 pad 1: /C13 -> /C6
- SW91 pad 1: /C13 -> /C7
- SW92 pad 1: /C7 -> /C8
- SW93 pad 1: /C8 -> /C9
- SW94 pad 1: /C9 -> /C10
- SW95 pad 1: /C10 -> /C11
- TP2 pad 1: 3.3VOUT -> 3.3VIN
Routing:
- net 5VIN: track 0.00 -> 555.3 mm
- net /L5: track 0.00 -> 441.4 mm, vias 0 -> 13
- net /L4: track 0.00 -> 391.0 mm, vias 0 -> 7
- net /L6: track 0.00 -> 380.9 mm, vias 0 -> 17
- net /L3: track 0.00 -> 363.3 mm, vias 0 -> 8
- net /L2: track 0.00 -> 346.6 mm, vias 0 -> 7
- net /L1: track 19.0 -> 360.8 mm, vias 0 -> 12
- net /C1: track 0.00 -> 338.6 mm, vias 0 -> 29
- net /C12: track 0.00 -> 328.4 mm, vias 0 -> 17
- net /L7: track 0.00 -> 326.5 mm, vias 0 -> 13
- net /C11: track 0.00 -> 321.5 mm, vias 0 -> 27
- net /C2: track 0.00 -> 300.0 mm, vias 0 -> 22
- net /C10: track 0.00 -> 281.3 mm, vias 0 -> 24
- net /C3: track 0.00 -> 273.6 mm, vias 0 -> 20
- net /C9: track 0.00 -> 240.9 mm, vias 0 -> 22
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- added copper zone on B.Cu, net 3.3VIN
- added copper zone on F.Cu, net 3.3VIN
- added copper zone on B.Cu, net GND
- added copper zone on F.Cu, net GND
Other:
- board outline added: 359.4 x 142.3 mm
- board text added: "MILLIEU : 135.825 mm"
