File: Électrique/Clavier/Clavier_drive_1/Clavier_drive_1.kicad_sch (KiCad schematic)
At the start: 176 parts, among them IC12 TCAN332DR, IC3 TLV1117-33IDCY, J16 B5B-XH-A_LF__SN_, J9 Conn_01x02_Pin, SW15 Switch, SW16 Switch, SW17 Switch, SW18 Switch, SW19 Switch, SW20 Switch, SW23 Switch, SW24 Switch, SW25 Switch, SW26 Switch, SW27 Switch, SW28 Switch, SW29 Switch, SW30 Switch, SW31 Switch, SW32 Switch, SW33 Switch, SW34 Switch, SW35 Switch, SW36 Switch, SW37 Switch, SW38 Switch, SW39 Switch, SW40 Switch, SW41 Switch, SW42 Switch, SW43 Switch, SW44 Switch, SW45 Switch, SW46 Switch, SW47 Switch, SW48 Switch, SW51 Switch, SW52 Switch, SW53 Switch, SW54 Switch, SW55 Switch, SW56 Switch, SW57 Switch, SW58 Switch, SW59 Switch, SW60 Switch, SW61 Switch, SW62 Switch, SW63 Switch, SW64 Switch, SW65 Switch, SW66 Switch, SW67 Switch, SW68 Switch, SW69 Switch, SW70 Switch, SW71 Switch, SW72 Switch, SW73 Switch, SW74 Switch, SW75 Switch, SW76 Switch, SW79 Switch, SW80 Switch, SW81 Switch, SW82 Switch, SW83 Switch, SW84 Switch, SW86 Switch, SW87 Switch, SW88 Switch, SW89 Switch, SW90 Switch, SW91 Switch, SW92 Switch, SW93 Switch, SW94 Switch, SW95 Switch

Commit message: ajout firmware + modif readme
Parts:
- removed D1, D2, D3, D35, D36, D4, D5, D6, D63, D64, D7: 1N4148W, Diode_SMD:D_SOD-123, symbol Diode:1N4148W
- removed J16: B5B-XH-A_LF__SN_, SamacSys:SHDR5W64P0X250_1X5_1490X575X700P, symbol SamacSys_Parts:B5B-XH-A_LF__SN_
- removed J9: Conn_01x02_Pin, SamacSys:SHDRRA2W50P0X200_1X2_600X770X525P, symbol SamacSys_Parts:B2B-XH-AM_LF__SN_
- removed S1, S2, S3, S4, S5, S6, S7: MTS-103, switchboard:MTS-103 Switch, symbol SamacSys_Parts:2MS1T1B3M2QES
- removed SW35, SW36, SW63, SW64: Switch, PCM_marbastlib-mx:SW_MX_HS_CPG151101S11_1u, symbol Switch:SW_Push
- added C101, C102, C139, C140, C141, C142, C143, C144: CL31A476MPHNNNE, SamacSys:CAPC3216X180N, symbol SamacSys_Parts:CL31A476MPHNNNE
- added C103, C104, C105, C106, C107, C108, C109, C110, C111, C112, C113, C114, C115, C116, C117, C118, C119, C120, C121, C122, C123, C124, C125, C126, C127, C128, C129, C130, C131, C132, C133, C134, C135, C136, C137, C138: 0.1uF, Capacitor_SMD:C_0402_1005Metric, symbol SamacSys_Parts:CC0603KRX7R9BB104
- added C2: 22uF, Capacitor_SMD:C_1206_3216Metric, symbol SamacSys_Parts:CL31A226KAHNNNE
- added D101, D102, D103, D105, D106, D107, D108, D109, D110, D111, D112, D113, D114: 1N4148W, Diode_SMD:D_SOD-123, symbol Diode:1N4148W
- added H101, H102, H103, H104, H105, H106, H107, H108, H109, H110, H111, H112: MountingHole, MountingHole:MountingHole_3.2mm_M3_DIN965, symbol Mechanical:MountingHole
- added IC101, IC102, IC104: SN74LVC1T45DBVR, SamacSys:SOT95P280X145-6N, symbol SamacSys_Parts:SN74LVC1T45DBVR
- added IC103: H11L1SR2VM, SamacSys:H11L1SR2VM, symbol SamacSys_Parts:H11L1SR2VM
- added J101, J102, J103, J104, J105, J106: SJ1-3533N, SamacSys:SJ13533N, symbol SamacSys_Parts:SJ1-3533N
- added LED101, LED102, LED103, LED104, LED105, LED106, LED107, LED108, LED109, LED110, LED111, LED112, LED113, LED114, LED115, LED116, LED117, LED118, LED119, LED120, LED121, LED122, LED123, LED124, LED125, LED126, LED127, LED128, LED129, LED130: SK6812MINI-E, JANKO:LED-SMD_4P-L3.2-W2.8-LS5.9_SK6812MINI-E, symbol JANKO:SK6812MINI-E_C5149201
- added Q1: AO3401A, Package_TO_SOT_SMD:SOT-23, symbol Transistor_FET:AO3401A
- added R101, R104: R510, Resistor_SMD:R_0603_1608Metric, symbol Device:R
- added R102, R103, R105, R106, R107: R220, Resistor_SMD:R_0603_1608Metric, symbol Device:R
- added R33: R1K, Resistor_SMD:R_0603_1608Metric, symbol Device:R
- added R34: 10k, Resistor_SMD:R_0603_1608Metric, symbol Device:R
- added S1: TS-1088-AR02016, SamacSys:TS1088AR02016, symbol SamacSys_Parts:TS-1088-AR02016
- added SW101, SW102, SW103, SW104, SW105, SW106, SW107, SW108, SW109, SW110, SW111, SW112: Switch, PCM_marbastlib-mx:SW_MX_HS_CPG151101S11_1u, symbol Switch:SW_Push
- R24: now fitted
- TP2: now left out of the parts list
Connections:
- net 3.3VOUT is gone; now on net 3.3VIN: C1.1, C8.1, D104.2 (A), IC3.2 (OUTPUT_2), IC3.4 (OUTPUT), TP2.1
- net RXD is gone; now on net RXD CAN: IC12.4 (RXD)
- net TXD is gone; now on net TXD CAN: IC12.1 (TXD)
- net 3.3VIN: now also Q1.3 (D)
- net 5VIN: now also C101.2, C102.2, C104.2, C105.1, C106.1, C107.1, C108.1, C109.1, C110.1, C111.1, C112.1, C113.1, C114.1, C115.1, C116.1, C117.1, C118.1, C119.1, C120.1, C121.1, C122.1, C123.1, C124.1, C125.1, C126.1, C127.1, C128.1, C130.2, C132.2, C133.1, C134.1, C135.1, C136.1, C137.1, C138.1, C139.2, C140.2, C141.2, C142.2, C143.2, C144.2, C2.1, IC101.6 (VCCB), IC102.6 (VCCB), IC104.6 (VCCB), J101.1 (SLEEVE), LED101.3 (VDD), LED102.3 (VDD), LED103.3 (VDD), LED104.3 (VDD), LED105.3 (VDD), LED106.3 (VDD), LED107.3 (VDD), LED108.3 (VDD), LED109.3 (VDD), LED110.3 (VDD), LED111.3 (VDD), LED112.3 (VDD), LED113.3 (VDD), LED114.3 (VDD), LED115.3 (VDD), LED116.3 (VDD), LED117.3 (VDD), LED118.3 (VDD), LED119.3 (VDD), LED120.3 (VDD), LED121.3 (VDD), LED122.3 (VDD), LED123.3 (VDD), LED124.3 (VDD), LED125.3 (VDD), LED126.3 (VDD), LED127.3 (VDD), LED128.3 (VDD), LED129.3 (VDD), LED130.3 (VDD), R103.2, R107.2
- net C1: now also A1.20 (GPIO15), SW103.1
- net C10: now also A1.24 (GPIO18), SW94.1, SW108.1; no longer SW95.1
- net C11: now also A1.22 (GPIO17), SW95.1, SW107.1
- net C12: now also A1.21 (GPIO16), SW112.1
- net C2: now also A1.19 (GPIO14), SW86.1, SW104.1
- net C3: now also A1.17 (GPIO13), SW87.1, SW105.1; no longer SW86.1
- net C4: now also A1.16 (GPIO12), SW88.1, SW106.1; no longer SW87.1
- net C5: now also A1.5 (GPIO3), SW89.1, SW102.1; no longer SW88.1
- net C6: now also A1.4 (GPIO2), SW90.1, SW101.1; no longer SW89.1
- net C7: now also A1.34 (GPIO28_ADC2), SW91.1, SW110.1; no longer SW92.1
- net C8: now also A1.32 (GPIO27_ADC1), SW92.1, SW111.1; no longer SW93.1
- net C9: now also A1.25 (GPIO19), SW93.1, SW109.1; no longer SW94.1
- net CAN+: now also J105.1 (SLEEVE), J106.1 (SLEEVE)
- net CAN-: now also J105.2 (TIP), J106.2 (TIP)
- net GND: now also A1.13 (GND), A1.18 (GND), A1.23 (GND), A1.28 (GND), A1.3 (GND), A1.38 (GND), A1.8 (GND), A1.D2 (GND), C101.1, C102.1, C103.1, C104.1, C105.2, C106.2, C107.2, C108.2, C109.2, C110.2, C111.2, C112.2, C113.2, C114.2, C115.2, C116.2, C117.2, C118.2, C119.2, C120.2, C121.2, C122.2, C123.2, C124.2, C125.2, C126.2, C127.2, C128.2, C129.1, C130.1, C131.1, C132.1, C133.2, C134.2, C135.2, C136.2, C137.2, C138.2, C139.1, C140.1, C141.1, C142.1, C143.1, C144.1, C2.2, IC101.2 (GND), IC102.2 (GND), IC103.5 (GND), IC104.2 (GND), J101.2 (TIP), J102.1 (SLEEVE), J104.1 (SLEEVE), LED101.1 (GND), LED102.1 (GND), LED103.1 (GND), LED104.1 (GND), LED105.1 (GND), LED106.1 (GND), LED107.1 (GND), LED108.1 (GND), LED109.1 (GND), LED110.1 (GND), LED111.1 (GND), LED112.1 (GND), LED113.1 (GND), LED114.1 (GND), LED115.1 (GND), LED116.1 (GND), LED117.1 (GND), LED118.1 (GND), LED119.1 (GND), LED120.1 (GND), LED121.1 (GND), LED122.1 (GND), LED123.1 (GND), LED124.1 (GND), LED125.1 (GND), LED126.1 (GND), LED127.1 (GND), LED128.1 (GND), LED129.1 (GND), LED130.1 (GND), R33.1
- net L1: now also A1.9 (GPIO6)
- net L2: now also A1.10 (GPIO7)
- net L3: now also A1.11 (GPIO8), D43.1 (K)
- net L4: now also A1.12 (GPIO9)
- net L5: now also A1.29 (GPIO22); no longer D91.1 (K)
- net L6: now also A1.27 (GPIO21), D91.1 (K)
- net L7: now also A1.26 (GPIO20), D102.1 (K), D103.1 (K), D105.1 (K), D106.1 (K), D107.1 (K), D108.1 (K), D109.1 (K), D110.1 (K), D111.1 (K), D112.1 (K), D113.1 (K), D114.1 (K)
- net RUN: now also A1.30 (RUN), R34.1, S1.1 (COM)
- net RXD CAN: now reaches A1.1 (GPIO0)
- net LED_DATA: now reaches A1.15 (GPIO11)
- net LED_DATA: now also IC101.3 (A)
- net TXD CAN: now reaches A1.2 (GPIO1)
- net 3.3V RP: now reaches A1.36 (3V3)
- net 3.3V RP: now also C103.2, C129.2, C131.2, IC101.1 (VCCA), IC101.5 (DIR), IC102.1 (VCCA), IC102.5 (DIR), IC103.6 (VCC), IC104.1 (VCCA), IC104.5 (DIR), R104.1, R34.2
- net at A1.39 (VSYS): now also Q1.2 (S)
- net at A1.40 (VBUS): now also Q1.1 (G)
- net TX PICO MIDI: now reaches A1.6 (GPIO4)
- net TX PICO MIDI: now also IC102.3 (A)
- net  RX PICO MIDI: now reaches A1.7 (GPIO5)
- net  RX PICO MIDI: now also IC103.4 (VO), IC104.3 (A), R104.2
- removed net C13: SW90.1, SW91.1
- new net: R33.2, S1.2 (NO)
- new net: D101.2 (A), IC103.2 (CATHODE), J103.2 (TIP)
- new net: J103.3 (RING), R106.1
- new net: LED101.2 (DIN), R101.1
- new net: IC101.4 (B), R101.2
- new net: LED105.4 (DOUT), LED106.2 (DIN)
- new net: LED106.4 (DOUT), LED107.2 (DIN)
- new net: LED128.4 (DOUT), LED129.2 (DIN)
- new net: LED129.4 (DOUT), LED130.2 (DIN)
- new net: D111.2 (A), SW109.2
- new net: D112.2 (A), SW110.2
- new net: D108.2 (A), SW106.2
- new net: D114.2 (A), SW112.2
- new net: LED117.4 (DOUT), LED118.2 (DIN)
- new net: LED118.4 (DOUT), LED119.2 (DIN)
- new net: LED107.4 (DOUT), LED108.2 (DIN)
- new net: LED103.4 (DOUT), LED104.2 (DIN)
- new net: LED104.4 (DOUT), LED105.2 (DIN)
- new net: J102.2 (TIP), R102.1
- new net: LED126.4 (DOUT), LED127.2 (DIN)
- new net: LED127.4 (DOUT), LED128.2 (DIN)
- new net: LED113.4 (DOUT), LED114.2 (DIN)
- new net: LED101.4 (DOUT), LED102.2 (DIN)
- new net: D107.2 (A), SW105.2
- new net: D102.2 (A), SW101.2
- new net: LED125.4 (DOUT), LED126.2 (DIN)
- new net: D110.2 (A), SW108.2
- new net: D109.2 (A), SW107.2
- new net: D103.2 (A), SW102.2
- new net: J104.2 (TIP), R105.1
- new net: LED114.4 (DOUT), LED115.2 (DIN)
- new net: LED115.4 (DOUT), LED116.2 (DIN)
- new net: D106.2 (A), SW104.2
- new net: D113.2 (A), SW111.2
- new net: LED110.4 (DOUT), LED111.2 (DIN)
- new net: LED111.4 (DOUT), LED112.2 (DIN)
- new net: LED121.4 (DOUT), LED122.2 (DIN)
- new net: LED122.4 (DOUT), LED123.2 (DIN)
- new net: J104.3 (RING), R107.1
- new net: LED109.4 (DOUT), LED110.2 (DIN)
- new net: D105.2 (A), SW103.2
- new net: LED119.4 (DOUT), LED120.2 (DIN)
- new net: LED120.4 (DOUT), LED121.2 (DIN)
- new net: LED102.4 (DOUT), LED103.2 (DIN)
- new net: LED116.4 (DOUT), LED117.2 (DIN)
- new net: LED108.4 (DOUT), LED109.2 (DIN)
- new net: LED123.4 (DOUT), LED124.2 (DIN)
- new net: J102.3 (RING), R103.1
- new net DOUT1: LED112.4 (DOUT), LED113.2 (DIN)
- new net DOUT2: LED124.4 (DOUT), LED125.2 (DIN)
- new net MIDI IN: D101.1 (K), IC103.1 (ANODE), R106.2
- new net THRU: IC104.4 (B), R105.2
- new net TX OUT: IC102.4 (B), R102.2
- no-connect marks 2 -> 19
Other:
- note added: "LED"
- note added: "MIDI IN"
- note added: "MIDI OUT"
- note added: "MIDI THRU"
- note removed: "FLASH"
- moved on the sheet: A1, C1, C10, C78, C8, C9, D104, D15, D16, D17, D18, D19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
