File: Électrique/Moteur/Solenoide_drive/Solenoide_drive.kicad_pcb (KiCad board)
At the start: 4 copper layers, 150 x 71 mm, 170 parts, among them IC1 SC1510_13_-A4, IC10 DRV8874PWPR, IC11 DRV8874PWPR, IC12 TCAN332DR, IC13 DRV8874PWPR, IC14 DRV8874PWPR, IC15 DRV8874PWPR, IC16 DRV8874PWPR, IC17 74HC4051D,653, IC18 74HC4051D,653, IC2 TPS54302DDCR, IC3 TLV1117-33IDCY, IC4 DRV8874PWPR, IC5 DRV8874PWPR, IC6 DRV8874PWPR, IC7 DRV8874PWPR, IC8 DRV8874PWPR, IC9 DRV8874PWPR, J1 Conn_01x02_Pin, J10 Conn_01x02_Pin, J11 1729128, J12 Conn_01x02_Pin, J13 Conn_01x02_Pin, J14 Conn_01x02_Pin, J15 Conn_01x02_Pin, J2 Conn_01x02_Pin, J3 Conn_01x02_Pin, J4 Conn_01x02_Pin, J5 Conn_01x02_Pin, J6 Conn_01x02_Pin, J7 Conn_01x02_Pin, J8 Conn_01x02_Pin, J9 Conn_01x02_Pin, Y1 ABM8-272-T3

Commit message: mises à jour photo readme2
Parts:
- removed IC18: 74HC4051D,653, SamacSys:74HC4051D653
- added C100: 10uF, Capacitor_SMD:C_1206_3216Metric, F.Cu at (97.7, 18.2)
- added C101: C680, EasyEDA:CAP-SMD_BD12.5-L13.0-W13.0-LS14.4-FD, F.Cu at (106.1, 17.5)
- added C102: C680, EasyEDA:CAP-SMD_BD12.5-L13.0-W13.0-LS14.4-FD, F.Cu at (119.8, 17.5)
- added J16: B5B-XH-A_LF__SN_, SamacSys:SHDR5W64P0X250_1X5_1490X575X700P, F.Cu at (89.4, 16.4)
- added J17: Conn_01x02_Pin, SamacSys:SHDRRA2W50P0X200_1X2_600X770X525P, F.Cu at (6.65, 9.00)
- added TP1: TestPoint, SamacSys:TestPoint_Pad_D1.0mm_Silkless, F.Cu at (23.1, 21.3)
- added TP2: TestPoint, SamacSys:TestPoint_Pad_D1.0mm_Silkless, F.Cu at (39.5, 11.0)
- added TP3: TestPoint, SamacSys:TestPoint_Pad_D1.0mm_Silkless, F.Cu at (54.0, 6.00)
- added TP4: TestPoint, SamacSys:TestPoint_Pad_D4.0mm_Silkless, F.Cu at (35.0, 2.80)
- added TP5: TestPoint, SamacSys:TestPoint_Pad_D4.0mm_Silkless, F.Cu at (75.0, 69.0)
- added TP6: TestPoint, SamacSys:TestPoint_Pad_D4.0mm_Silkless, F.Cu at (147.0, 9.20)
- added TP7: TestPoint, SamacSys:TestPoint_Pad_D4.0mm_Silkless, F.Cu at (2.90, 19.4)
- C10, C14, C15, C16, C17, C18, C19, C2, C20, C21, C22, C23, C24, C25, C26, C29, C3, C33, C35, C37, C39, C42, C45, C46, C48, C50, C51, C54, C56, C58, C60, C62, C63, C66, C68, C70, C73, C74, C75, C78, C8, C82, C83, C84, C85, C86, C87, C88, C89, C98, C99: footprint SamacSys:CAPC1608X90N -> Capacitor_SMD:C_0402_1005Metric
- D1: value SMCJ28A -> SMCJ26CAHE3_A/H
- F1: value 0451010.MRL -> 0458010.DR; footprint SamacSys:0451010MRL -> SamacSys:FUSC3216X158N
- IC17: value 74HC4051D,653 -> 74HC4067PW,118; footprint SamacSys:74HC4051D653 -> SamacSys:SOP65P640X110-24N
- moved D1 61.3 mm to (130.1, 18.0)
- moved F1 60.6 mm to (135.7, 21.4), turned to 0 degrees
- moved C99 16.1 mm to (76.2, 15.1), turned to -90 degrees
- moved IC17 13.4 mm to (69.9, 7.00), turned to -90 degrees
- moved C98 3.77 mm to (73.4, 11.9), turned to -90 degrees
- moved R2 2.96 mm to (15.9, 23.4)
- moved L1 2.96 mm to (16.9, 14.7)
- moved C3 2.96 mm to (13.7, 19.8)
- moved C6 2.96 mm to (20.2, 21.7)
- moved C7 2.96 mm to (10.5, 20.3)
- moved R1 2.96 mm to (13.7, 22.5)
- moved R3 2.96 mm to (20.2, 24.7)
- moved R4 2.96 mm to (20.2, 23.2)
- moved R5 2.96 mm to (20.2, 20.2)
- moved C4 2.96 mm to (23.9, 13.6)
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Connections:
- net CANH renamed CAN+
- net CANL renamed CAN-
- C99 pad 1: 3.3VIN -> /RUN
- F1 pad 1: Net-(F1-Pad1) -> 24VIN
- F1 pad 2: 24VIN -> Net-(F1-Pad2)
- IC1 pad 1: unconnected-(IC1-GPIO4-Pad1) -> /FAULT2
- IC1 pad 11: unconnected-(IC1-GPIO12-Pad11) -> /FAULT4
- IC1 pad 12: unconnected-(IC1-GPIO13-Pad12) -> /SENS4
- IC1 pad 13: unconnected-(IC1-GPIO14-Pad13) -> /PWM5
- IC1 pad 14: unconnected-(IC1-GPIO15-Pad14) -> /nSLEEP
- IC1 pad 16: unconnected-(IC1-GPIO16-Pad16) -> /FAULT7
- IC1 pad 17: unconnected-(IC1-GPIO17-Pad17) -> /FAULT6
- IC1 pad 18: unconnected-(IC1-GPIO18-Pad18) -> /PWM7
- IC1 pad 19: unconnected-(IC1-GPIO19-Pad19) -> /SENS7
- IC1 pad 2: unconnected-(IC1-GPIO5-Pad2) -> /PWM2
- IC1 pad 20: unconnected-(IC1-GPIO20-Pad20) -> /PWM6
- IC1 pad 21: unconnected-(IC1-GPIO21-Pad21) -> /SENS6
- IC1 pad 22: unconnected-(IC1-GPIO22-Pad22) -> /FAULT9
- IC1 pad 23: unconnected-(IC1-GPIO23-Pad23) -> /PWM9
- IC1 pad 25: unconnected-(IC1-GPIO24-Pad25) -> /SENS9
- IC1 pad 26: unconnected-(IC1-GPIO25-Pad26) -> /FAULT8
- IC1 pad 27: unconnected-(IC1-GPIO26-Pad27) -> /PWM8
- IC1 pad 28: unconnected-(IC1-GPIO27-Pad28) -> /SENS8
- IC1 pad 3: unconnected-(IC1-GPIO6-Pad3) -> /SENS2
- IC1 pad 33: unconnected-(IC1-SWCLK-Pad33) -> /SDCLK
- IC1 pad 34: unconnected-(IC1-SWDIO-Pad34) -> /SWDIO
- IC1 pad 35: unconnected-(IC1-RUN-Pad35) -> /RUN
- IC1 pad 36: unconnected-(IC1-GPIO28-Pad36) -> /FAULT11
- IC1 pad 37: unconnected-(IC1-GPIO29-Pad37) -> /PWM11
- IC1 pad 38: unconnected-(IC1-GPIO30-Pad38) -> /SENS11
- IC1 pad 39: unconnected-(IC1-GPIO31-Pad39) -> /FAULT10
- IC1 pad 4: unconnected-(IC1-GPIO7-Pad4) -> /PWM3
- IC1 pad 40: unconnected-(IC1-GPIO32-Pad40) -> /PWM10
- IC1 pad 42: unconnected-(IC1-GPIO33-Pad42) -> /SENS10
- IC1 pad 44: unconnected-(IC1-GPIO35-Pad44) -> /PWM0
- IC1 pad 45: unconnected-(IC1-GPIO36-Pad45) -> /S3
- IC1 pad 46: unconnected-(IC1-GPIO37-Pad46) -> /FAULT1
- IC1 pad 47: unconnected-(IC1-GPIO38-Pad47) -> /S2
- IC1 pad 48: unconnected-(IC1-GPIO39-Pad48) -> /FAULT0
- IC1 pad 49: /MUX2OUT -> unconnected-(IC1-GPIO40_ADC0-Pad49)
- IC1 pad 53: unconnected-(IC1-GPIO42_ADC2-Pad53) -> /MUX_EN
- IC1 pad 54: unconnected-(IC1-GPIO43_ADC3-Pad54) -> /S1
- IC1 pad 55: /MUX1OUT -> /S0
- IC1 pad 56: unconnected-(IC1-GPIO45_ADC5-Pad56) -> /MUX OUT
- IC1 pad 57: unconnected-(IC1-GPIO46_ADC6-Pad57) -> /RXD
- IC1 pad 58: unconnected-(IC1-GPIO47_ADC7-Pad58) -> /TXD
- IC1 pad 6: unconnected-(IC1-GPIO8-Pad6) -> /SENS3
- IC1 pad 7: unconnected-(IC1-GPIO9-Pad7) -> /SENS5
- IC1 pad 77: unconnected-(IC1-GPIO0-Pad77) -> /SENS0
- IC1 pad 78: unconnected-(IC1-GPIO1-Pad78) -> /PWM1
- IC1 pad 79: unconnected-(IC1-GPIO2-Pad79) -> /SENS1
- IC1 pad 8: unconnected-(IC1-GPIO10-Pad8) -> /FAULT5
- IC1 pad 80: unconnected-(IC1-GPIO3-Pad80) -> /FAULT3
- IC1 pad 81: unconnected-(IC1-GND-Pad81) -> GND
- IC1 pad 9: unconnected-(IC1-GPIO11-Pad9) -> /PWM4
- IC17 pad 1: /ADC4 -> /MUX OUT
- IC17 pad 10: /S1 -> /S0
- IC17 pad 11: /S0 -> /S1
- IC17 pad 12: /ADC3 -> GND
- IC17 pad 13: /ADC0 -> /S3
- IC17 pad 14: /ADC1 -> /S2
- IC17 pad 15: /ADC2 -> /MUX_EN
- IC17 pad 16: 3.3VIN -> unconnected-(IC17-Y15-Pad16)
- IC17 pad 3: /MUX1OUT -> /ADC11
- IC17 pad 4: unconnected-(IC17-Y7-Pad4) -> /ADC8
- IC17 pad 5: /ADC5 -> /ADC10
- IC17 pad 6: /MUX_EN -> /ADC9
- IC17 pad 7: GND -> /ADC7
- IC17 pad 8: GND -> /ADC6
- IC17 pad 9: /S2 -> unconnected-(IC17-Y0-Pad9)
- J11 pad 1: Net-(F1-Pad1) -> Net-(F1-Pad2)
Routing:
- net 3.3VIN: track 507.4 -> 894.1 mm, vias 43 -> 47
- net /ADC0: track 11.5 -> 165.9 mm, vias 1 -> 4
- net CAN+: track 1.87 -> 142.6 mm
- net CAN-: track 1.87 -> 142.5 mm
- net /ADC1: track 11.6 -> 142.4 mm, vias 1 -> 4
- net /ADC6: track 11.7 -> 140.8 mm, vias 1 -> 6
- net /ADC2: track 11.5 -> 138.6 mm, vias 1 -> 6
- net /PWM11: track 1.48 -> 121.3 mm, vias 1 -> 2
- net /SENS11: track 1.36 -> 120.9 mm, vias 1 -> 2
- net /FAULT11: track 11.9 -> 127.7 mm, vias 1 -> 2
- net /ADC7: track 11.5 -> 121.5 mm, vias 1 -> 6
- net /ADC11: track 11.5 -> 118.9 mm, vias 1 -> 2
- net /SENS10: track 1.36 -> 107.0 mm, vias 1 -> 2
- net /PWM10: track 1.48 -> 102.7 mm, vias 1 -> 2
- net /ADC3: track 11.4 -> 111.5 mm, vias 1 -> 4
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- added copper zone on B.Cu, net GND
- added copper zone on F.Cu, net Net-(F1-Pad2)
- removed copper zone on F.Cu, net Net-(F1-Pad1)
Other:
- board size 150 x 71 mm -> 150 x 71.5 mm
- board text added: "1.1V"
- board text added: "24V"
- board text added: "3.3V"
- board text added: "3.3VIN"
- board text added: "5V"
- board text added: "CAN+"
- board text added: "CAN-"
- board text added: "GND"
- board text added: "PWM0"
- board text added: "PWM1"
- board text added: "PWM10"
- board text added: "PWM11"
- board text added: "PWM2"
- board text added: "PWM3"
- board text added: "PWM4"
- board text added: "PWM5"
- board text added: "PWM6"
- board text added: "PWM7"
- board text added: "PWM8"
- board text added: "PWM9"
- board text added: "RDX"
- board text added: "RUN"
- board text added: "SDLCK"
- board text added: "SWDIO"
- board text added: "TDX"

Commit message: ajout firmware + modif readme
Parts:
- added C103: EEE-FK1H100P, SamacSys:EEE1AA101SP, F.Cu at (5.60, 19.2)
- added C104: 0.1uF, Capacitor_SMD:C_0402_1005Metric, F.Cu at (96.3, 5.10)
- added FB1: BLM18PG121SN1D, SamacSys:BLM18SP221SN1B, F.Cu at (5.60, 25.4)
- added R33: R1K, Resistor_SMD:R_0603_1608Metric, F.Cu at (86.0, 9.40)
- added R34: 10k, Resistor_SMD:R_0603_1608Metric, F.Cu at (78.1, 6.12)
- added R35: R1K, Resistor_SMD:R_0603_1608Metric, F.Cu at (89.0, 9.40)
- added R36: 10k, Resistor_SMD:R_0603_1608Metric, F.Cu at (95.8, 7.10)
- added S1: TS-1088-AR02016, SamacSys:TS1088AR02016, F.Cu at (83.8, 6.20)
- added S2: TS-1088-AR02016, SamacSys:TS1088AR02016, F.Cu at (91.3, 6.20)
- J16: value B5B-XH-A_LF__SN_ -> B4B-XH-A_LF__SN_; footprint SamacSys:SHDR5W64P0X250_1X5_1490X575X700P -> SamacSys:B4BXHALFSN
- L1: footprint SamacSys:INDPM6965X300N -> SamacSys:SRP6060FA4R7M
- TP7: footprint SamacSys:TestPoint_Pad_D4.0mm_Silkless -> SamacSys:TestPoint_Pad_D1.0mm_Silkless
- moved TP7 45.2 mm to (46.3, 6.70)
- moved C99 9.85 mm to (79.5, 5.82)
- moved C7 2.83 mm to (10.6, 23.1), turned to -90 degrees
- moved F1 2.20 mm to (137.9, 21.4)
- moved D1 2.01 mm to (132.1, 17.8)
- moved C102 1.70 mm to (121.5, 17.5)
- moved C9 1.52 mm to (25.9, 20.5)
- moved C101 1.00 mm to (107.1, 17.5)
- moved C100 0.80 mm to (98.5, 18.2)
- moved L1 0.75 mm to (16.2, 14.7), turned to 90 degrees
- turned J16 to 180 degrees
Connections:
- C2 pad 1: 24VIN -> Net-(C103-+)
- C7 pad 1: 24VIN -> Net-(C103-+)
- IC1 pad 43: unconnected-(IC1-GPIO34-Pad43) -> /Bouton test
- IC1 pad 52: unconnected-(IC1-GPIO41_ADC1-Pad52) -> /FREQ OSC
- IC2 pad 3: 24VIN -> Net-(C103-+)
- R1 pad 1: 24VIN -> Net-(C103-+)
- TP7 pad 1: GND -> /FREQ OSC
Routing:
- net /Bouton test: track 0.00 -> 44.0 mm, vias 0 -> 2
- net 3.3VIN: track 894.1 -> 860.0 mm
- net /nSLEEP: track 352.9 -> 377.6 mm
- net GND: track 100.0 -> 114.6 mm, vias 619 -> 626
- net Net-(C103-+): track 0.00 -> 12.8 mm
- net /FREQ OSC: track 0.00 -> 12.4 mm, vias 0 -> 2
- net /RUN: track 26.5 -> 37.5 mm
- net 24VIN: track 45.8 -> 41.0 mm
- net Net-(S2-NO): track 0.00 -> 3.47 mm
- net Net-(S1-NO): track 0.00 -> 3.47 mm
- net 5VIN: track 57.8 -> 54.9 mm
- net /ADC9: track 102.5 -> 99.7 mm
- net /ADC7: track 121.5 -> 119.1 mm
- net /ADC6: track 140.8 -> 138.5 mm
- net /ADC8: track 77.8 -> 76.0 mm
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- added copper zone on B.Cu, net Net-(F1-Pad2)
Other:
- board text added: "TEST"
