File: Électrique/Moteur/Solenoide_drive/Solenoide_drive.kicad_sch (KiCad schematic)
At the start: 170 parts, among them IC1 SC1510_13_-A4, IC10 DRV8874PWPR, IC11 DRV8874PWPR, IC12 TCAN332DR, IC13 DRV8874PWPR, IC14 DRV8874PWPR, IC15 DRV8874PWPR, IC16 DRV8874PWPR, IC17 74HC4051D,653, IC18 74HC4051D,653, IC2 TPS54302DDCR, IC3 TLV1117-33IDCY, IC4 DRV8874PWPR, IC5 DRV8874PWPR, IC6 DRV8874PWPR, IC7 DRV8874PWPR, IC8 DRV8874PWPR, IC9 DRV8874PWPR, J1 Conn_01x02_Pin, J10 Conn_01x02_Pin, J11 1729128, J12 Conn_01x02_Pin, J13 Conn_01x02_Pin, J14 Conn_01x02_Pin, J15 Conn_01x02_Pin, J2 Conn_01x02_Pin, J3 Conn_01x02_Pin, J4 Conn_01x02_Pin, J5 Conn_01x02_Pin, J6 Conn_01x02_Pin, J7 Conn_01x02_Pin, J8 Conn_01x02_Pin, J9 Conn_01x02_Pin, Y1 ABM8-272-T3

Commit message: mises à jour photo readme2
Parts:
- removed F1: 0451010.MRL, SamacSys:0451010MRL, symbol SamacSys_Parts:0451010.MRL
- removed IC17, IC18: 74HC4051D,653, 74HC4051D653, symbol SamacSys_Parts:74HC4051D,653
- added C100: 10uF, Capacitor_SMD:C_1206_3216Metric, symbol SamacSys_Parts:CL31A106KBHNNNE
- added C101, C102: C680, EasyEDA:CAP-SMD_BD12.5-L13.0-W13.0-LS14.4-FD, symbol SamacSys_Parts:470U_50V_RVT1H471M1213
- added F1: 0458010.DR, FUSC3216X158N, symbol SamacSys_Parts:0458010.DR
- added IC17: 74HC4067PW,118, SamacSys:SOP65P640X110-24N, symbol SamacSys_Parts:74HC4067PW,118
- added J16: B5B-XH-A_LF__SN_, SamacSys:SHDR5W64P0X250_1X5_1490X575X700P, symbol SamacSys_Parts:B5B-XH-A_LF__SN_
- added J17: Conn_01x02_Pin, SamacSys:SHDRRA2W50P0X200_1X2_600X770X525P, symbol SamacSys_Parts:B2B-XH-AM_LF__SN_
- added TP1, TP2, TP3: TestPoint, SamacSys:TestPoint_Pad_D1.0mm_Silkless, symbol Connector:TestPoint
- added TP4, TP5, TP6, TP7: TestPoint, SamacSys:TestPoint_Pad_D4.0mm_Silkless, symbol Connector:TestPoint
- C10, C14, C15, C16, C17, C18, C19, C2, C20, C21, C22, C23, C24, C25, C26, C29, C3, C33, C35, C37, C39, C42, C45, C46, C48, C50, C51, C54, C56, C58, C60, C62, C63, C66, C68, C70, C73, C74, C75, C78, C8, C82, C83, C84, C85, C86, C87, C88, C89, C98, C99: footprint SamacSys:CAPC1608X90N -> Capacitor_SMD:C_0402_1005Metric
- D1: value SMCJ28A -> SMCJ26CAHE3_A/H
Connections:
- net MUX1OUT is gone; now on net S0: IC1.55 (GPIO44_ADC4)
- net +1V1: now also TP3.1
- net 24VIN: now also C100.1, C101.1, C102.1, F1.1
- net 3.3VIN: now also IC17.24 (VCC), J16.2, TP2.1; no longer C99.1
- net 5VIN: now also J17.1, TP1.1
- net ADC0: now also IC17.22 (Y9)
- net ADC1: now also IC17.21 (Y10)
- net ADC10: now also IC17.5 (Y4)
- net ADC11: now also IC17.3 (Y6)
- net ADC2: now also IC17.20 (Y11)
- net ADC3: now also IC17.19 (Y12)
- net ADC4: now also IC17.18 (Y13)
- net ADC5: now also IC17.17 (Y14)
- net ADC6: now also IC17.8 (Y1)
- net ADC7: now also IC17.7 (Y2)
- net ADC8: now also IC17.4 (Y5)
- net ADC9: now also IC17.6 (Y3)
- net FAULT0: now also IC1.48 (GPIO39)
- net FAULT1: now also IC1.46 (GPIO37)
- net FAULT10: now also IC1.39 (GPIO31)
- net FAULT11: now also IC1.36 (GPIO28)
- net FAULT2: now also IC1.1 (GPIO4)
- net FAULT3: now also IC1.80 (GPIO3)
- net FAULT4: now also IC1.11 (GPIO12)
- net FAULT5: now also IC1.8 (GPIO10)
- net FAULT6: now also IC1.17 (GPIO17)
- net FAULT7: now also IC1.16 (GPIO16)
- net FAULT8: now also IC1.26 (GPIO25)
- net FAULT9: now also IC1.22 (GPIO22)
- net GND: now also IC1.81 (GND), C100.2, C101.2, C102.2, IC17.12 (GND), J16.1, J17.2, TP4.1, TP5.1, TP6.1, TP7.1
- net MUX_EN: now also IC1.53 (GPIO42_ADC2), IC17.15 (~{E})
- net PWM0: now also IC1.44 (GPIO35)
- net PWM1: now also IC1.78 (GPIO1)
- net PWM10: now also IC1.40 (GPIO32)
- net PWM11: now also IC1.37 (GPIO29)
- net PWM2: now also IC1.2 (GPIO5)
- net PWM3: now also IC1.4 (GPIO7)
- net PWM4: now also IC1.9 (GPIO11)
- net PWM5: now also IC1.13 (GPIO14)
- net PWM6: now also IC1.20 (GPIO20)
- net PWM7: now also IC1.18 (GPIO18)
- net PWM8: now also IC1.27 (GPIO26)
- net PWM9: now also IC1.23 (GPIO23)
- net RXD: now also IC1.57 (GPIO46_ADC6)
- net S0: now also IC17.10 (S0)
- net S1: now also IC1.54 (GPIO43_ADC3), IC17.11 (S1)
- net S2: now also IC1.47 (GPIO38), IC17.14 (S2)
- net SENS0: now also IC1.77 (GPIO0)
- net SENS1: now also IC1.79 (GPIO2)
- net SENS10: now also IC1.42 (GPIO33)
- net SENS11: now also IC1.38 (GPIO30)
- net SENS2: now also IC1.3 (GPIO6)
- net SENS3: now also IC1.6 (GPIO8)
- net SENS4: now also IC1.12 (GPIO13)
- net SENS5: now also IC1.7 (GPIO9)
- net SENS6: now also IC1.21 (GPIO21)
- net SENS7: now also IC1.19 (GPIO19)
- net SENS8: now also IC1.28 (GPIO27)
- net SENS9: now also IC1.25 (GPIO24)
- net TXD: now also IC1.58 (GPIO47_ADC7)
- net nSLEEP: now also IC1.14 (GPIO15)
- net at J11.1: now also F1.2
- net SDCLK: now reaches IC1.33 (SWCLK)
- net SDCLK: now also J16.3
- net SWDIO: now reaches IC1.34 (SWDIO)
- net SWDIO: now also J16.4
- net RUN: now reaches IC1.35 (RUN)
- net RUN: now also C99.1, J16.5
- net S3: now reaches IC1.45 (GPIO36)
- net S3: now also IC17.13 (S3)
- net MUX OUT: now reaches IC1.56 (GPIO45_ADC5)
- net MUX OUT: now also IC17.1 (Z)
- net CANH renamed CAN+
- net CANL renamed CAN-
- net MUX2OUT: no longer names the net of IC1.49 (GPIO40_ADC0)
- no-connect marks 6 -> 17
Other:
- note added: "Alim + protection + bulk"
- note added: "FLASH"
- note added: "Sortie alim pour la carte clavier"
- note added: "Tests points"
- moved on the sheet: C1, C10, C16, C19, C2, C23, C3, C4, C5, C6, C7, C76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

Commit message: ajout firmware + modif readme
Parts:
- removed J16: B5B-XH-A_LF__SN_, SamacSys:SHDR5W64P0X250_1X5_1490X575X700P, symbol SamacSys_Parts:B5B-XH-A_LF__SN_
- added C103: EEE-FK1H100P, EEE1AA101SP, symbol SamacSys_Parts:EEE-FK1H100P
- added C104: 0.1uF, Capacitor_SMD:C_0402_1005Metric, symbol SamacSys_Parts:CC0603KRX7R9BB104
- added FB1: BLM18PG121SN1D, BLM18SP221SN1B, symbol SamacSys_Parts:BLM18PG121SN1D
- added J16: B4B-XH-A_LF__SN_, B4BXHALFSN, symbol SamacSys_Parts:B4B-XH-A_LF__SN_
- added R33, R35: R1K, Resistor_SMD:R_0603_1608Metric, symbol Device:R
- added R34, R36: 10k, Resistor_SMD:R_0603_1608Metric, symbol Device:R
- added S1, S2: TS-1088-AR02016, TS1088AR02016, symbol SamacSys_Parts:TS-1088-AR02016
- L1: footprint SamacSys:INDPM6965X300N -> SRP6060FA4R7M; symbol SamacSys_Parts:IHLP2525CZER100M11 -> SamacSys_Parts:SRP6060FA-100M; Manufacturer_Name Vishay -> Bourns; Manufacturer_Part_Number IHLP2525CZER100M11 -> SRP6060FA-100M; Mouser Part Number 70-IHLP2525CZER100M1 -> 652-SRP6060FA-100M; Mouser Price/Stock https://www.mouser.co.uk/ProductDetail/Vishay-Dale/IHLP2525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 -> https://www.mouser.co.uk/ProductDetail/Bourns/SRP6060FA-100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
- TP1, TP2, TP3, TP4, TP5, TP6: now left out of the parts list
- TP7: footprint SamacSys:TestPoint_Pad_D4.0mm_Silkless -> SamacSys:TestPoint_Pad_D1.0mm_Silkless; now left out of the parts list
Connections:
- net 24VIN: now also FB1.1; no longer C2.1, C7.1, IC2.3 (VIN), R1.1
- net 3.3VIN: now also J16.2, R34.2, R36.2
- net GND: now also C103.2 (-), C104.2, J16.1, R33.1, R35.1; no longer TP7.1
- net RUN: now also R34.1, S1.1 (COM)
- net SDCLK: now also J16.3
- net SWDIO: now also J16.4
- net Bouton test: now reaches IC1.43 (GPIO34)
- net Bouton test: now also C104.1, R36.1, S2.1 (COM)
- net FREQ OSC: now reaches IC1.52 (GPIO41_ADC1)
- net FREQ OSC: now also TP7.1
- new net: R33.2, S1.2 (NO)
- new net: C103.1 (+), C2.1, C7.1, FB1.2, IC2.3 (VIN), R1.1
- new net: R35.2, S2.2 (NO)
- no-connect marks 17 -> 15
